File: PCB/macro-attempt-2.kicad_pcb (KiCad board)
At the start: 2 copper layers, 54.2 x 59.1 mm, 24 parts

Commit message: savepoint
Parts:
- moved LED_R 1.90 mm to (200.6, 144.8)
- moved R4 1.90 mm to (210.1, 134.8)
- moved R7 1.90 mm to (166.6, 135.2)
- moved MX1 1.90 mm to (166.7, 102.1)
- moved MX8 1.90 mm to (185.8, 102.1)
- moved MX9 1.90 mm to (204.8, 102.1)
- moved R12 1.90 mm to (200.7, 148.2)
- moved R6 1.90 mm to (164.5, 116.1)
- moved R9 1.90 mm to (204.8, 97.0)
- moved ESP32S1 1.90 mm to (199.7, 102.2)
- moved MX2 1.90 mm to (185.8, 121.2)
- moved MX5 1.90 mm to (204.8, 121.2)
- moved MX6 1.90 mm to (166.7, 121.2)
- moved R1 1.90 mm to (161.1, 96.9)
- moved R2 1.90 mm to (188.4, 113.0)
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Other:
- board size 54.2 x 59.1 mm -> 64 x 64 mm
